File: steno_half.kicad_pcb (KiCad board)
At the start: 2 copper layers, 144 x 90.8 mm, 38 parts, among them J1 IDC-Header_2x05_P2.54mm_Verti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, J2 IDC-Header_2x05_P2.54mm_Verti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

Commit message: Primeiro roteamento OK, sem erros de DRC. Adicionando também diretório com o footprint que fiz do STM 32 Blue Pill.
Parts:
- renumbered REF** to H1, REF** to H2, REF** to H3, REF** to H4, REF** to H5, REF** to H6, REF** to H7
Routing:
- net R1: track 0.00 -> 255.2 mm, vias 0 -> 2
- net C5: track 0.00 -> 209.3 mm
- net R0: track 0.00 -> 208.4 mm, vias 0 -> 2
- net C4: track 0.00 -> 171.7 mm
- net C3: track 0.00 -> 151.8 mm, vias 0 -> 1
- net C2: track 0.00 -> 132.4 mm
- net C1: track 0.00 -> 114.6 mm, vias 0 -> 1
- net C0: track 0.00 -> 100.7 mm, vias 0 -> 1
- net C6: track 0.00 -> 100.4 mm
- net X7: track 0.00 -> 51.7 mm
- net X9: track 0.00 -> 42.7 mm, vias 0 -> 1
- net X6: track 0.00 -> 39.8 mm
- net X8: track 0.00 -> 36.1 mm
- net X1: track 0.00 -> 36.0 mm
- net X10: track 0.00 -> 34.2 mm
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